File: samples/gerber/gerber.kicad_sch (KiCad schematic)
At the start: 7 parts, among them J1 USB_C_Receptacle_USB2.0_16P, J2 Conn_01x04_Socket, U1 W25Q16JVSS

Commit message: sample/gerber: add rotated footprint
Parts:
- added J3: USB_C_Receptacle_USB2.0_16P, Connector_USB:USB_C_Receptacle_G-Switch_GT-USB-7051x, symbol Connector:USB_C_Receptacle_USB2.0_16P
Connections:
- net GND: now also J1.A1 (GND), J1.A12 (GND), J1.B1 (GND), J1.B12 (GND), J1.S1 (SHIELD), J3.A1 (GND), J3.A12 (GND), J3.B1 (GND), J3.B12 (GND), J3.S1 (SHIELD)
- net V: now also J3.A4 (VBUS), J3.A9 (VBUS), J3.B4 (VBUS), J3.B9 (VBUS)
- no-connect marks 8 -> 12

Commit message: gerber: handle kicad exported filenames
Parts:
- added C3: C, Capacitor_SMD:C_1210_3225Metric, symbol Device:C
- added J4: USB_C_Receptacle_USB2.0_16P, Connector_USB:USB_C_Receptacle_G-Switch_GT-USB-7051x, symbol Connector:USB_C_Receptacle_USB2.0_16P
Connections:
- net GND: now also C3.2, J4.A1 (GND), J4.A12 (GND), J4.B1 (GND), J4.B12 (GND), J4.S1 (SHIELD)
- net V: now also C3.1, J4.A4 (VBUS), J4.A9 (VBUS), J4.B4 (VBUS), J4.B9 (VBUS)
- no-connect marks 12 -> 18

Commit message: update gerber samples
Parts:
- J1, J3, J4: LCSC (none) -> C2843970
Changed lines of the file:
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@@
+			)
+		)
+		(property "LCSC" "C2843970"
+			(at 59.69 119.38 0)
+			(effects
+				(font
+					(size 1.27 1.27)
+				)
+				(hide yes)
 			)
 		)
@@
 			)
 		)
+		(property "LCSC" "C2843970"
+			(at 101.6 77.47 0)
+			(effects
+				(font
+					(size 1.27 1.27)
+				)
+				(hide yes)
+			)
+		)
 		(pin "B7"
 		)
@@
 			(at 106.68 160.02 0)
 			(effects
+				(font
+					(size 1.27 1.27)
+				)
+				(hide yes)
+			)
+		)
+		(property "LCSC" "C2843970"
+			(at 106.68 160.02 0)
+			(effects
