File: samples/maze_radius.kicad_pcb (KiCad board)
At the start: 2 copper layers, 38 x 38 mm, 0 parts

Commit message: add/update samples/{/maze,maze_radius}.kicad_pcb
Other:
- board text added: "a=-30 r=0.5"
- board text added: "a=-30 r=1.25"
- board text added: "a=-30 r=2"
- board text added: "a=30 r=0.25"
- board text added: "a=30 r=1"
- board text added: "a=30 r=1.75"
- board text removed: "a=30 r=0"
Changed lines of the file:
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@@
 		)
 	)
-	(gr_text "a=30 r=0"
+	(gr_text "a=30 r=0.25"
 		(at 104 130 270)
 		(layer "User.4")
@@
 		)
 	)
-	(gr_text "a=-30 r=0"
+	(gr_text "a=-30 r=0.5"
 		(at 107 130 270)
 		(layer "User.4")
@@
 		)
 	)
-	(gr_text "a=30 r=0"
+	(gr_text "a=30 r=1"
 		(at 110 130 270)
 		(layer "User.4")
@@
 		)
 	)
-	(gr_text "a=-30 r=0"
+	(gr_text "a=-30 r=1.25"
 		(at 113 130 270)
 		(layer "User.4")
@@
 		)
 	)
-	(gr_text "a=30 r=0"
+	(gr_text "a=30 r=1.75"
 		(at 116 130 270)
 		(layer "User.4")
@@
 		)
 	)
-	(gr_text "a=-30 r=0"
+	(gr_text "a=-30 r=2"
 		(at 119 130 270)
 		(layer "User.4")
