File: samples/maze_radius_fan.kicad_pcb (KiCad board)
At the start: 2 copper layers, 38 x 38 mm, 0 parts

Commit message: update samples/maze_radius_fan.kicad_pcb
Other:
- board text added: "a=-15 r=0.15"
- board text added: "a=-70 r=0.7"
- board text added: "a=15 r=0.15"
- board text added: "a=70 r=0.7"
- board text removed: "a=-10 r=0.1"
- board text removed: "a=-5 r=0"
- board text removed: "a=10 r=0.1"
- board text removed: "a=5 r=0"
Changed lines of the file:
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@@
 	(gr_line
 		(start 90 90)
-		(end 100 130)
+		(end 130 100)
 		(stroke
 			(width 0.1)
@@
 	(gr_line
 		(start 90 95)
-		(end 97.5 130)
+		(end 130 102.5)
 		(stroke
 			(width 0.1)
@@
 	(gr_line
 		(start 90 100)
-		(end 95 130)
+		(end 130 105)
+		(stroke
+			(width 0.1)
+			(type solid)
+		)
+		(layer "User.4")
+	)
+	(gr_line
+		(start 90 105)
+		(end 130 107.5)
+		(stroke
+			(width 0.1)
+			(type solid)
+		)
+		(layer "User.4")
+	)
+	(gr_line
+		(start 90 108.75)
+		(end 130 108.75)
+		(stroke
+			(width 0.1)
+			(type solid)
+		)
+		(layer "User.4")
+	)
+	(gr_line
+		(start 90 111.25)
+		(end 130 111.25)
+		(stroke
+			(width 0.1)
+			(type solid)
+		)
+		(layer "User.4")
+	)
+	(gr_line
+		(start 90 115)
+		(end 130 112.5)
+		(stroke
+			(width 0.1)
+			(type solid)
+		)
+		(layer "User.4")
+	)
+	(gr_line
+		(start 90 120)
+		(end 130 115)
+		(stroke
+			(width 0.1)
+			(type solid)
+		)
+		(layer "User.4")
+	)
+	(gr_line
+		(start 90 125)
+		(end 130 117.5)
+		(stroke
+			(width 0.1)
+			(type solid)
+		)
+		(layer "User.4")
+	)
+	(gr_line
+		(start 90 130)
+		(end 130 120)
 		(stroke
 			(width 0.1)
@@
 	(gr_line
 		(start 95 90)
-		(end 102.5 130)
+		(end 130 97.5)
+		(stroke
+			(width 0.1)
+			(type solid)
+		)
+		(layer "User.4")
+	)
+	(gr_line
+		(start 95 130)
+		(end 130 122.5)
 		(stroke
 			(width 0.1)
@@
 	(gr_line
 		(start 100 90)
-		(end 105 130)
-		(stroke
-			(width 0.1)
-			(type solid)
-		)
-		(layer "User.4")
-	)
-	(gr_line
-		(start 105 90)
-		(end 107.5 130)
-		(stroke
-			(width 0.1)
-			(type solid)
-		)
-		(layer "User.4")
-	)
-	(gr_line
-		(start 108.75 90)
-		(end 108.75 130)
-		(stroke
-			(width 0.1)
-			(type solid)
-		)
-		(layer "User.4")
-	)
-	(gr_line
-		(start 111.25 90)
-		(end 111.25 130)
-		(stroke
-			(width 0.1)
-			(type solid)
-		)
-		(layer "User.4")
-	)
-	(gr_line
-		(start 115 90)
-		(end 112.5 130)
-		(stroke
-			(width 0.1)
-			(type solid)
-		)
-		(layer "User.4")
-	)
-	(gr_line
-		(start 120 90)
-		(end 115 130)
-		(stroke
-			(width 0.1)
-			(type solid)
-		)
-		(layer "User.4")
-	)
-	(gr_line
-		(start 125 90)
-		(end 117.5 130)
-		(stroke
-			(width 0.1)
-			(type solid)
-		)
-		(layer "User.4")
-	)
-	(gr_line
-		(start 130 90)
-		(end 120 130)
-		(stroke
-			(width 0.1)
-			(type solid)
-		)
-		(layer "User.4")
-	)
-	(gr_line
-		(start 130 95)
-		(end 122.5 130)
-		(stroke
-			(width 0.1)
-			(type solid)
-		)
-		(layer "User.4")
-	)
-	(gr_line
-		(start 130 100)
-		(end 125 130)
-		(stroke
-			(width 0.1)
-			(type solid)
-		)
-		(layer "User.4")
+		(end 130 95)
+		(stroke
+			(width 0.1)
+			(type solid)
+		)
+		(layer "User.4")
+	)
+	(gr_line
+		(start 100 130)
+		(end 130 125)
+		(stroke
+			(width 0.1)
+			(type solid)
+		)
+		(layer "User.4")
+	)
+	(gr_text "a=70 r=0.7"
+		(at 130 95 0)
+		(layer "User.4")
+		(effects
+			(font
+				(size 1 1)
+				(thickness 0.1)
+			)
+			(justify left bottom)
+		)
 	)
 	(gr_text "a=-60 r=0.6"
-		(at 95 130 270)
+		(at 130 97.5 0)
 		(layer "User.4")
 		(effects
@@
 	)
 	(gr_text "a=50 r=0.5"
-		(at 97.5 130 270)
+		(at 130 100 0)
 		(layer "User.4")
 		(effects
@@
 	)
 	(gr_text "a=-40 r=0.4"
-		(at 100 130 270)
+		(at 130 102.5 0)
 		(layer "User.4")
 		(effects
@@
 	)
 	(gr_text "a=30 r=0.3"
-		(at 102.5 130 270)
+		(at 130 105 0)
 		(layer "User.4")
 		(effects
@@
 	)
 	(gr_text "a=-20 r=0.2"
-		(at 105 130 270)
-		(layer "User.4")
-		(effects
-			(font
-				(size 1 1)
-				(thickness 0.1)
-			)
-			(justify left bottom)
-		)
-	)
-	(gr_text "a=10 r=0.1"
-		(at 107.5 130 270)
-		(layer "User.4")
-		(effects
-			(font
-				(size 1 1)
-				(thickness 0.1)
-			)
-			(justify left bottom)
-		)
-	)
-	(gr_text "a=-10 r=0.1"
-		(at 112.5 130 270)
+		(at 130 107.5 0)
 		(layer "User.4")
 		(effects
@@
 	)
 	(gr_text "a=20 r=0.2"
-		(at 115 130 270)
+		(at 130 112.5 0)
 		(layer "User.4")
 		(effects
@@
 	)
 	(gr_text "a=-30 r=0.3"
-		(at 117.5 130 270)
+		(at 130 115 0)
 		(layer "User.4")
 		(effects
@@
 	)
 	(gr_text "a=40 r=0.4"
-		(at 120 130 270)
+		(at 130 117.5 0)
 		(layer "User.4")
 		(effects
@@
 	)
 	(gr_text "a=-50 r=0.5"
-		(at 122.5 130 270)
+		(at 130 120 0)
 		(layer "User.4")
 		(effects
@@
 	)
 	(gr_text "a=60 r=0.6"
-		(at 125 130 270)
-		(layer "User.4")
-		(effects
-			(font
-				(size 1 1)
-				(thickness 0.1)
-			)
-			(justify left bottom)
-		)
-	)
-	(gr_text "a=-5 r=0"
-		(at 108.75 130 270)
+		(at 130 122.5 0)
+		(layer "User.4")
+		(effects
+			(font
+				(size 1 1)
+				(thickness 0.1)
+			)
+			(justify left bottom)
+		)
+	)
+	(gr_text "a=-70 r=0.7"
+		(at 130 125 0)
+		(layer "User.4")
+		(effects
+			(font
+				(size 1 1)
+				(thickness 0.1)
+			)
+			(justify left bottom)
+		)
+	)
+	(gr_text "a=15 r=0.15"
+		(at 130 108.75 0)
 		(layer "User.4")
 		(effects
@@
 		)
 	)
-	(gr_text "a=5 r=0"
-		(at 111.25 130 270)
-		(layer "User.4")
-		(effects
+	(gr_text "a=-15 r=0.15"
+		(at 130 111.25 0)
+		(layer "User.4")
+		(effects
