File: samples/assembly-power.kicad_pcb (KiCad board)
At the start: 4 copper layers, 29.4 x 22.1 mm, 6 parts, among them J2 Conn_01x06_Pin, J3 Conn_01x06_Socket

Commit message: update assembly samples
Parts:
- moved led 0.48 mm to (135.8, 76.5)
Changed lines of the file:
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@@
 	(footprint "Kikakuka:CouplerFixed"
 		(layer "F.Cu")
-		(at 135.34 76.5 90)
+		(at 135.82 76.5 90)
 		(property "Reference" "led"
 			(at 0 0 90)
@@
 			)
 		)
-		(property "Z" "2.7"
+		(property "Z" "3"
 			(at 0 0 153)
 			(unlocked yes)
