File: samples/assembly-power.kicad_pcb (KiCad board)
At the start: 4 copper layers, 29.4 x 22.1 mm, 6 parts, among them J2 Conn_01x06_Pin, J3 Conn_01x06_Socket

Commit message: Update assembly coupler samples
Parts:
- led, mcu, mezzanine: footprint Kikakuka:CouplerFixed -> PCM_Kikakuka:CouplerFixed
Changed lines of the file:
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@@
 		)
 	)
-	(footprint "Kikakuka:CouplerFixed"
+	(footprint "PCM_Kikakuka:CouplerFixed"
 		(layer "F.Cu")
 		(at 138.76 69.873728 27)
@@
 			)
 		)
-		(property "Description" ""
+		(property "Description" "Fixed FreekiCAD alignment plane. Matches a CouplerMoving footprint with the same reference. Z moves along the PCB surface normal; positive Offset moves on the PCB surface in the triangle direction; Tilt rotates around local X. Unitless lengths default to mm; mm/in/mil/um are supported."
 			(at 0 0 27)
 			(unlocked yes)
@@
 			)
 		)
-		(property "Z" "4.4mm"
-			(at 0 0 90)
+		(property "Z" "4.4 mm"
+			(at 0 0 27)
 			(unlocked yes)
 			(layer "F.Fab")
@@
 		)
 		(property "Offset" "0 mm"
-			(at 0 0 90)
+			(at 0 0 27)
+			(unlocked yes)
+			(layer "F.Fab")
+			(hide yes)
+			(effects
+				(font
+					(size 1 1)
+					(thickness 0.15)
+				)
+			)
+		)
+		(property "Tilt" "0"
+			(at 0 0 27)
 			(unlocked yes)
 			(layer "F.Fab")
@@
 		)
 		(fp_line
+			(start -0.25 -0.25)
+			(end 0.25 -0.25)
+			(stroke
+				(width 0.1)
+				(type default)
+			)
+			(layer "Cmts.User")
+		)
+		(fp_line
+			(start 0 -0.5)
+			(end 0 0)
+			(stroke
+				(width 0.1)
+				(type default)
+			)
+			(layer "Cmts.User")
+		)
+		(fp_line
 			(start 0 0)
 			(end -1 -1)
@@
 		(embedded_fonts no)
 	)
-	(footprint "Kikakuka:CouplerFixed"
+	(footprint "PCM_Kikakuka:CouplerFixed"
 		(layer "F.Cu")
 		(at 135.82 76.5 90)
@@
 		)
 		(property "Value" "CouplerFixed"
-			(at -0.000001 1 90)
+			(at 0 1 90)
 			(unlocked yes)
 			(layer "F.Fab")
@@
 			)
 		)
-		(property "Description" ""
+		(property "Description" "Fixed FreekiCAD alignment plane. Matches a CouplerMoving footprint with the same reference. Z moves along the PCB surface normal; positive Offset moves on the PCB surface in the triangle direction; Tilt rotates around local X. Unitless lengths default to mm; mm/in/mil/um are supported."
 			(at 0 0 90)
 			(unlocked yes)
@@
 			)
 		)
-		(property "Z" "3"
-			(at 0 0 153)
+		(property "Z" "3 mm"
+			(at 0 0 90)
 			(unlocked yes)
 			(layer "F.Fab")
@@
 		)
 		(property "Offset" "0 mm"
-			(at 0 0 153)
+			(at 0 0 90)
 			(unlocked yes)
 			(layer "F.Fab")
@@
 		)
 		(property "Tilt" "90"
-			(at 0 0 0)
+			(at 0 0 90)
 			(unlocked yes)
 			(layer "F.Fab")
@@
 			(start -1 -1)
 			(end 1 -1)
+			(stroke
+				(width 0.1)
+				(type default)
+			)
+			(layer "Cmts.User")
+		)
+		(fp_line
+			(start 0 -0.5)
+			(end 0 0)
+			(stroke
+				(width 0.1)
+				(type default)
+			)
+			(layer "Cmts.User")
+		)
+		(fp_line
+			(start -0.25 -0.25)
+			(end 0.25 -0.25)
 			(stroke
 				(width 0.1)
@@
 		)
 	)
-	(footprint "Kikakuka:CouplerFixed"
+	(footprint "PCM_Kikakuka:CouplerFixed"
 		(layer "B.Cu")
 		(at 123.1 76.47 180)
@@
 			)
 		)
-		(property "Description" ""
+		(property "Description" "Fixed FreekiCAD alignment plane. Matches a CouplerMoving footprint with the same reference. Z moves along the PCB surface normal; positive Offset moves on the PCB surface in the triangle direction; Tilt rotates around local X. Unitless lengths default to mm; mm/in/mil/um are supported."
 			(at 0 0 0)
 			(unlocked yes)
@@
 			)
 		)
-		(property "Z" "5.6"
+		(property "Z" "5.6 mm"
 			(at 0 0 0)
 			(unlocked yes)
@@
 		)
 		(fp_line
+			(start 0 0.5)
+			(end 0 0)
+			(stroke
+				(width 0.1)
+				(type default)
+			)
+			(layer "Cmts.User")
+		)
+		(fp_line
 			(start 0 0)
 			(end -1 1)
 			(stroke
 				(width 0.1)
+				(type default)
+			)
+			(layer "Cmts.User")
+		)
+		(fp_line
+			(start -0.25 0.25)
+			(end 0.25 0.25)
+			(stroke
+				(width 0.1)
