File: samples/fpc.kicad_pcb (KiCad board)
At the start: 2 copper layers, 15.1 x 13.2 mm, 5 parts, among them J1 Conn_01x02_Pin

Commit message: Align couplers after flex PCB bending
Parts:
- added J2: Conn_01x02_Pin, Connector_PinHeader_1.00mm:PinHeader_1x02_P1.00mm_Horizontal, F.Cu at (92.3, 97.3)
- added conn: CouplerFixed, Kikakuka:CouplerFixed, F.Cu at (91.1, 97.3)
Other:
- board size 15.1 x 13.2 mm -> 15.1 x 15 mm

Commit message: update sample/{fpc,fpc2}
Parts:
- moved J2 0.56 mm to (91.8, 97.3)
- moved conn 0.56 mm to (90.5, 97.3)
Changed lines of the file:
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@@
 		(capping no)
 		(filling no)
-		(zone_defaults)
 		(pcbplotparams
 			(layerselection 0x00000000_00000000_55555555_5755f5ff)
@@
 	(footprint "Kikakuka:CouplerFixed"
 		(layer "F.Cu")
-		(at 91.1 97.33 -90)
+		(at 90.54 97.33 -90)
 		(property "Reference" "conn"
 			(at 0 0 270)
@@
 	(footprint "Connector_PinHeader_1.00mm:PinHeader_1x02_P1.00mm_Horizontal"
 		(layer "F.Cu")
-		(at 92.35 97.33 180)
+		(at 91.79 97.33 180)
 		(descr "Through hole angled pin header, 1x02, 1.00mm pitch, 2.0mm pin length, single row")
 		(tags "Through hole angled pin header THT 1x02 1.00mm single row")

Commit message: Add CouplerOrigin to FPC sample
Parts:
- added REF**: CouplerOrigin, Kikakuka:CouplerOrigin, F.Cu at (97.9, 89.7)
Changed lines of the file:
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@@
+		(embedded_fonts no)
+	)
+	(footprint "Kikakuka:CouplerOrigin"
+		(layer "F.Cu")
+		(at 97.917 89.662)
+		(property "Reference" "REF**"
+			(at 0 0 0)
+			(unlocked yes)
+			(layer "Dwgs.User")
+			(hide yes)
+			(effects
+				(font
+					(size 1 1)
+					(thickness 0.1)
+				)
+			)
+		)
+		(property "Value" "CouplerOrigin"
+			(at 0 1 0)
+			(unlocked yes)
+			(layer "F.Fab")
+			(hide yes)
+			(effects
+				(font
+					(size 1 1)
+					(thickness 0.15)
+				)
+			)
+		)
+		(property "Datasheet" ""
+			(at 0 0 0)
+			(unlocked yes)
+			(layer "F.Fab")
+			(hide yes)
+			(effects
+				(font
+					(size 1 1)
+					(thickness 0.15)
+				)
+			)
+		)
+		(property "Description" ""
+			(at 0 0 0)
+			(unlocked yes)
+			(layer "F.Fab")
+			(hide yes)
+			(effects
+				(font
+					(size 1 1)
+					(thickness 0.15)
+				)
+			)
+		)
+		(property "Z" "0 mm"
+			(at 0 0 0)
+			(unlocked yes)
+			(layer "F.Fab")
+			(hide yes)
+			(effects
+				(font
+					(size 1 1)
+					(thickness 0.15)
+				)
+			)
+		)
+		(property "Tilt" "0"
+			(at 0 0 0)
+			(unlocked yes)
+			(layer "F.Fab")
+			(hide yes)
+			(effects
+				(font
+					(size 1 1)
+					(thickness 0.15)
+				)
+			)
+		)
+		(attr smd)
+		(duplicate_pad_numbers_are_jumpers no)
+		(fp_line
+			(start -1 -1)
+			(end 1 -1)
+			(stroke
+				(width 0.1)
+				(type default)
+			)
+			(layer "Cmts.User")
+		)
+		(fp_line
+			(start 0 0)
+			(end -1 -1)
+			(stroke
+				(width 0.1)
+				(type default)
+			)
+			(layer "Cmts.User")
+		)
+		(fp_line
+			(start 1 -1)
+			(end 0 0)
+			(stroke
+				(width 0.1)
+				(type default)
+			)
+			(layer "Cmts.User")
+		)
+		(fp_circle
+			(center 0 -0.5)
+			(end 0 -0.75)
+			(stroke
+				(width 0.1)
+				(type default)
+			)
+			(fill no)
+			(layer "Cmts.User")
+		)
 		(embedded_fonts no)
 	)
